Commit message: 240723

File: urdf/pai_2_12_240723.urdf (robot description, URDF)
Before this commit: robot pai_2_12_240715, 13 links, 12 joints
Links:
- removed link l_ankle_link
- removed link l_foot_link
- removed link l_kuan2_link
- removed link l_kuan_link
- removed link r_ankle_link
- removed link r_foot_link
- removed link r_kuan2_link
- removed link r_kuan_link
- added link l_ankle_pitch_link, mass 0.01180204; collision mesh filename=package://pai_2_12_240723/meshes/l_ankle_pitch_link.STL; visual mesh filename=package://pai_2_12_240723/meshes/l_ankle_pitch_link.STL
- added link l_ankle_roll_link, mass 0.18592619; collision mesh filename=package://pai_2_12_240723/meshes/l_ankle_roll_link.STL; visual mesh filename=package://pai_2_12_240723/meshes/l_ankle_roll_link.STL
- added link l_hip_roll_link, mass 0.75405217; collision mesh filename=package://pai_2_12_240723/meshes/l_hip_roll_link.STL; visual mesh filename=package://pai_2_12_240723/meshes/l_hip_roll_link.STL
- added link l_hip_yaw_link, mass 0.40825297; collision mesh filename=package://pai_2_12_240723/meshes/l_hip_yaw_link.STL; visual mesh filename=package://pai_2_12_240723/meshes/l_hip_yaw_link.STL
- added link r_ankle_pitch_link, mass 0.01180204; collision mesh filename=package://pai_2_12_240723/meshes/r_ankle_pitch_link.STL; visual mesh filename=package://pai_2_12_240723/meshes/r_ankle_pitch_link.STL
- added link r_ankle_roll_link, mass 0.18592619; collision mesh filename=package://pai_2_12_240723/meshes/r_ankle_roll_link.STL; visual mesh filename=package://pai_2_12_240723/meshes/r_ankle_roll_link.STL
- added link r_hip_roll_link, mass 0.75405217; collision mesh filename=package://pai_2_12_240723/meshes/r_hip_roll_link.STL; visual mesh filename=package://pai_2_12_240723/meshes/r_hip_roll_link.STL
- added link r_hip_yaw_link, mass 0.40825297; collision mesh filename=package://pai_2_12_240723/meshes/r_hip_yaw_link.STL; visual mesh filename=package://pai_2_12_240723/meshes/r_hip_yaw_link.STL
- link base_link: mass 0.767987723282303 -> 1.767987723282303; geometry collision mesh filename=package://pai_2_12_240723/meshes/base_link.STL; visual mesh filename=package://pai_2_12_240723/meshes/base_link.STL
- link l_calf_link: geometry collision mesh filename=package://pai_2_12_240723/meshes/l_calf_link.STL; visual mesh filename=package://pai_2_12_240723/meshes/l_calf_link.STL
- link l_thigh_link: geometry collision mesh filename=package://pai_2_12_240723/meshes/l_thigh_link.STL; visual mesh filename=package://pai_2_12_240723/meshes/l_thigh_link.STL
- link r_calf_link: geometry collision mesh filename=package://pai_2_12_240723/meshes/r_calf_link.STL; visual mesh filename=package://pai_2_12_240723/meshes/r_calf_link.STL
- link r_thigh_link: geometry collision mesh filename=package://pai_2_12_240723/meshes/r_thigh_link.STL; visual mesh filename=package://pai_2_12_240723/meshes/r_thigh_link.STL
Joints:
- removed joint l_ankle_joint
- removed joint l_foot_joint
- removed joint l_kuan2_joint
- removed joint l_kuan_joint
- removed joint r_ankle_joint
- removed joint r_foot_joint
- removed joint r_kuan2_joint
- removed joint r_kuan_joint
- added joint l_ankle_pitch_joint: type revolute, parent l_calf_link, child l_ankle_pitch_link, origin xyz=0 0 -0.17495 rpy=0 0 0, axis 0 -1 0, limit lower=-3.14 upper=3.14 effort=21 velocity=21
- added joint l_ankle_roll_joint: type revolute, parent l_ankle_pitch_link, child l_ankle_roll_link, origin xyz=0 0 0 rpy=0 0 0, axis -1 0 0, limit lower=-3.14 upper=3.14 effort=21 velocity=21
- added joint l_hip_roll_joint: type revolute, parent l_hip_yaw_link, child l_hip_roll_link, origin xyz=0 0 -0.056 rpy=0 0 0, axis 1 0 0, limit lower=-3.14 upper=3.14 effort=21 velocity=21
- added joint l_hip_yaw_joint: type revolute, parent base_link, child l_hip_yaw_link, origin xyz=-0.003125 0.075 -0.009 rpy=0 0 0, axis 0 0 1, limit lower=-3.14 upper=3.14 effort=21 velocity=21
- added joint r_ankle_pitch_joint: type revolute, parent r_calf_link, child r_ankle_pitch_link, origin xyz=0 0 -0.17495 rpy=0 0 0, axis 0 -1 0, limit lower=-3.14 upper=3.14 effort=21 velocity=21
- added joint r_ankle_roll_joint: type revolute, parent r_ankle_pitch_link, child r_ankle_roll_link, origin xyz=0 0 0 rpy=0 0 0, axis -1 0 0, limit lower=-3.14 upper=3.14 effort=21 velocity=21
- added joint r_hip_roll_joint: type revolute, parent r_hip_yaw_link, child r_hip_roll_link, origin xyz=0 0 -0.056 rpy=0 0 0, axis 1 0 0, limit lower=-3.14 upper=3.14 effort=21 velocity=21
- added joint r_hip_yaw_joint: type revolute, parent base_link, child r_hip_yaw_link, origin xyz=-0.003125 -0.075 -0.009 rpy=0 0 0, axis 0 0 1, limit lower=-3.14 upper=3.14 effort=21 velocity=21
- joint l_calf_joint: origin xyz=0.00750000000000105 0 -0.149812382665786 rpy=0 0 0 -> xyz=0.0075 0 -0.149812382665786 rpy=0 0 0
- joint l_thigh_joint: parent l_kuan2_link -> l_hip_roll_link
- joint r_calf_joint: origin xyz=0.00750000000000106 0 -0.149812382665787 rpy=0 0 0 -> xyz=0.0075 0 -0.149812382665786 rpy=0 0 0
- joint r_thigh_joint: parent r_kuan2_link -> r_hip_roll_link

Commit message: 修改了限位与初始位置

File: urdf/pai_2_12_240723.urdf (robot description, URDF)
Before this commit: robot pai_2_12_240723, 13 links, 12 joints
Joints:
- joint l_ankle_pitch_joint: axis 0 -1 0 -> 0 1 0; limit lower=-3.14 upper=3.14 effort=21 velocity=21 -> lower=-0.83 upper=0.59 effort=21 velocity=21
- joint l_ankle_roll_joint: axis -1 0 0 -> 1 0 0; limit lower=-3.14 upper=3.14 effort=21 velocity=21 -> lower=-0.4 upper=0.4 effort=21 velocity=21
- joint l_calf_joint: limit lower=-3.14 upper=3.14 effort=21 velocity=21 -> lower=0.0 upper=2.37 effort=21 velocity=21
- joint l_hip_roll_joint: limit lower=-3.14 upper=3.14 effort=21 velocity=21 -> lower=-0.22 upper=0.4 effort=21 velocity=21
- joint l_hip_yaw_joint: limit lower=-3.14 upper=3.14 effort=21 velocity=21 -> lower=-0.6 upper=0.6 effort=21 velocity=21
- joint l_thigh_joint: axis 0 -1 0 -> 0 1 0; limit lower=-3.14 upper=3.14 effort=21 velocity=21 -> lower=-2.25 upper=0.4 effort=21 velocity=21
- joint r_ankle_pitch_joint: axis 0 -1 0 -> 0 1 0; limit lower=-3.14 upper=3.14 effort=21 velocity=21 -> lower=-0.83 upper=0.59 effort=21 velocity=21
- joint r_ankle_roll_joint: axis -1 0 0 -> 1 0 0; limit lower=-3.14 upper=3.14 effort=21 velocity=21 -> lower=-0.4 upper=0.4 effort=21 velocity=21
- joint r_calf_joint: limit lower=-3.14 upper=3.14 effort=21 velocity=21 -> lower=0.0 upper=2.37 effort=21 velocity=21; origin xyz=0.0075 0 -0.149812382665786 rpy=0 0 0 -> xyz=0.0075 0 -0.149812382665786 rpy=0 -0.05009 0
- joint r_hip_roll_joint: limit lower=-3.14 upper=3.14 effort=21 velocity=21 -> lower=-0.4 upper=0.22 effort=21 velocity=21
- joint r_hip_yaw_joint: limit lower=-3.14 upper=3.14 effort=21 velocity=21 -> lower=-0.6 upper=0.6 effort=21 velocity=21
- joint r_thigh_joint: axis 0 -1 0 -> 0 1 0; limit lower=-3.14 upper=3.14 effort=21 velocity=21 -> lower=-2.25 upper=0.4 effort=21 velocity=21; origin xyz=0 0 0 rpy=0 0 0 -> xyz=0 0 0 rpy=0 0.05009 0
