Commit message: 修改了collision属性

File: urdf/pai_2_12_240723_rl.urdf (robot description, URDF)
Before this commit: robot pai_2_12_240723, 13 links, 12 joints
Links:
- link base_link: geometry collision box size=0.2 0.08 0.08; visual mesh filename=../meshes/base_link.STL
- link l_ankle_pitch_link: geometry collision box size=0.01 0.01 0.01; visual mesh filename=../meshes/l_ankle_pitch_link.STL
- link l_ankle_roll_link: geometry collision mesh filename=../meshes/l_ankle_roll_link.STL; visual mesh filename=../meshes/l_ankle_roll_link.STL
- link l_calf_link: geometry collision box size=0.03 0.035 0.12; visual mesh filename=../meshes/l_calf_link.STL
- link l_hip_roll_link: geometry collision box size=0.01 0.01 0.01; visual mesh filename=../meshes/l_hip_roll_link.STL
- link l_hip_yaw_link: geometry collision box size=0.01 0.01 0.01; visual mesh filename=../meshes/l_hip_yaw_link.STL
- link l_thigh_link: geometry collision box size=0.02 0.02 0.12; visual mesh filename=../meshes/l_thigh_link.STL
- link r_ankle_pitch_link: geometry collision box size=0.01 0.01 0.01; visual box size=0.01 0.01 0.01
- link r_ankle_roll_link: geometry collision mesh filename=../meshes/r_ankle_roll_link.STL; visual mesh filename=../meshes/r_ankle_roll_link.STL
- link r_calf_link: geometry collision box size=0.03 0.035 0.12; visual mesh filename=../meshes/r_calf_link.STL
- link r_hip_roll_link: geometry collision box size=0.01 0.01 0.01; visual mesh filename=../meshes/r_hip_roll_link.STL
- link r_hip_yaw_link: geometry collision box size=0.01 0.01 0.01; visual mesh filename=../meshes/r_hip_yaw_link.STL
- link r_thigh_link: geometry collision box size=0.02 0.02 0.12; visual box size=0.02 0.02 0.12
Joints:
- joint l_calf_joint: origin xyz=0.0075 0 -0.149812382665786 rpy=0 0 0 -> xyz=0.0075 0 -0.149812382665786 rpy=0 -0.05009 0
- joint l_thigh_joint: origin xyz=0 0 0 rpy=0 0 0 -> xyz=0 0 0 rpy=0 0.05009 0

Commit message: 修改了collision标签,增加了rl专用urdf

File: urdf/pai_2_12_240723_rl.urdf (robot description, URDF)
Before this commit: robot pai_2_12_240723, 13 links, 12 joints
Links:
- link base_link: geometry collision box size=0.2 0.08 0.08; visual mesh filename=../meshes/base_link.STL
- link l_ankle_pitch_link: geometry collision box size=0.01 0.01 0.01; visual mesh filename=../meshes/l_ankle_pitch_link.STL
- link l_ankle_roll_link: geometry collision mesh filename=../meshes/l_ankle_roll_link.STL; visual mesh filename=../meshes/l_ankle_roll_link.STL
- link l_calf_link: geometry collision box size=0.03 0.035 0.12; visual mesh filename=../meshes/l_calf_link.STL
- link l_hip_roll_link: geometry collision box size=0.01 0.01 0.01; visual mesh filename=../meshes/l_hip_roll_link.STL
- link l_hip_yaw_link: geometry collision box size=0.01 0.01 0.01; visual mesh filename=../meshes/l_hip_yaw_link.STL
- link l_thigh_link: geometry collision box size=0.02 0.02 0.12; visual mesh filename=../meshes/l_thigh_link.STL
- link r_ankle_roll_link: geometry collision mesh filename=../meshes/r_ankle_roll_link.STL; visual mesh filename=../meshes/r_ankle_roll_link.STL
- link r_calf_link: geometry collision box size=0.03 0.035 0.12; visual mesh filename=../meshes/r_calf_link.STL
- link r_hip_roll_link: geometry collision box size=0.01 0.01 0.01; visual mesh filename=../meshes/r_hip_roll_link.STL
- link r_hip_yaw_link: geometry collision box size=0.01 0.01 0.01; visual mesh filename=../meshes/r_hip_yaw_link.STL

Commit message: 修复文件

File: urdf/pai_2_12_240723_rl.urdf (robot description, URDF)
Before this commit: robot pai_2_12_240723, 13 links, 12 joints
Links:
- link r_thigh_link: geometry collision box size=0.02 0.02 0.12; visual mesh filename=../meshes/l_thigh_link.STL
Joints:
- joint l_ankle_roll_joint: axis 1 0 0 -> 1 0 0.0
