Commit message: first_commit

File: urdf/hi_1_21_240815.urdf (robot description, URDF)
Before this commit: robot hi_1_18_240815, 22 links, 21 joints
Links:
- link base_link: geometry collision mesh filename=package://hi_1_21_240815/meshes/base_link.STL; visual mesh filename=package://hi_1_21_240815/meshes/base_link.STL
- link l_ankle_pitch_link: geometry collision mesh filename=package://hi_1_21_240815/meshes/l_ankle_pitch_link.STL; visual mesh filename=package://hi_1_21_240815/meshes/l_ankle_pitch_link.STL
- link l_ankle_roll_link: geometry collision mesh filename=package://hi_1_21_240815/meshes/l_ankle_roll_link.STL; visual mesh filename=package://hi_1_21_240815/meshes/l_ankle_roll_link.STL
- link l_calf_link: geometry collision box size=0.03 0.035 0.12; visual mesh filename=package://hi_1_21_240815/meshes/l_calf_link.STL
- link l_elbow_roll_link: geometry collision mesh filename=package://hi_1_21_240815/meshes/l_elbow_roll_link.STL; visual mesh filename=package://hi_1_21_240815/meshes/l_elbow_roll_link.STL
- link l_elbow_yaw_link: geometry collision mesh filename=package://hi_1_21_240815/meshes/l_elbow_yaw_link.STL; visual mesh filename=package://hi_1_21_240815/meshes/l_elbow_yaw_link.STL
- link l_hip_roll_link: geometry collision box size=0.01 0.01 0.01; visual mesh filename=package://hi_1_21_240815/meshes/l_hip_roll_link.STL
- link l_hip_yaw_link: geometry collision box size=0.01 0.01 0.01; visual mesh filename=package://hi_1_21_240815/meshes/l_hip_yaw_link.STL
- link l_shoulder_pitch_link: geometry collision mesh filename=package://hi_1_21_240815/meshes/l_shoulder_pitch_link.STL; visual mesh filename=package://hi_1_21_240815/meshes/l_shoulder_pitch_link.STL
- link l_shoulder_roll_link: geometry collision mesh filename=package://hi_1_21_240815/meshes/l_shoulder_roll_link.STL; visual mesh filename=package://hi_1_21_240815/meshes/l_shoulder_roll_link.STL
- link l_thigh_link: geometry collision box size=0.02 0.02 0.12; visual mesh filename=package://hi_1_21_240815/meshes/l_thigh_link.STL
- link r_ankle_pitch_link: geometry collision mesh filename=package://hi_1_21_240815/meshes/r_ankle_pitch_link.STL; visual mesh filename=package://hi_1_21_240815/meshes/r_ankle_pitch_link.STL
- link r_ankle_roll_link: geometry collision mesh filename=package://hi_1_21_240815/meshes/r_ankle_roll_link.STL; visual mesh filename=package://hi_1_21_240815/meshes/r_ankle_roll_link.STL
- link r_calf_link: geometry collision box size=0.03 0.035 0.12; visual mesh filename=package://hi_1_21_240815/meshes/r_calf_link.STL
- link r_elbow_roll_link: geometry collision mesh filename=package://hi_1_21_240815/meshes/r_elbow_roll_link.STL; visual mesh filename=package://hi_1_21_240815/meshes/r_elbow_roll_link.STL
- link r_elbow_yaw_link: geometry collision mesh filename=package://hi_1_21_240815/meshes/r_elbow_yaw_link.STL; visual mesh filename=package://hi_1_21_240815/meshes/r_elbow_yaw_link.STL
- link r_hip_roll_link: geometry collision box size=0.01 0.01 0.01; visual mesh filename=package://hi_1_21_240815/meshes/r_hip_roll_link.STL
- link r_hip_yaw_link: geometry collision box size=0.01 0.01 0.01; visual mesh filename=package://hi_1_21_240815/meshes/r_hip_yaw_link.STL
- link r_shoulder_pitch_link: geometry collision mesh filename=package://hi_1_21_240815/meshes/r_shoulder_pitch_link.STL; visual mesh filename=package://hi_1_21_240815/meshes/r_shoulder_pitch_link.STL
- link r_shoulder_roll_link: geometry collision mesh filename=package://hi_1_21_240815/meshes/r_shoulder_roll_link.STL; visual mesh filename=package://hi_1_21_240815/meshes/r_shoulder_roll_link.STL
- link r_thigh_link: geometry collision box size=0.02 0.02 0.12; visual mesh filename=package://hi_1_21_240815/meshes/r_thigh_link.STL
- link waist_yaw_link: geometry collision mesh filename=package://hi_1_21_240815/meshes/waist_yaw_link.STL; visual mesh filename=package://hi_1_21_240815/meshes/waist_yaw_link.STL
