Commit message: fixed inertial

File: urdf/pai_cl_12_240823.urdf (robot description, URDF)
Before this commit: robot pai_cl_12_240823, 13 links, 12 joints
Links:
- removed link l_hip_yaw_link
- removed link r_hip_yaw_link
- added link l_hip_pitch_link, mass 0.37475; collision mesh filename=package://pai_cl_12_240823/meshes/l_hip_pitch_link.STL; visual mesh filename=package://pai_cl_12_240823/meshes/l_hip_pitch_link.STL
- added link r_hip_pitch_link, mass 0.37475; collision mesh filename=package://pai_cl_12_240823/meshes/r_hip_pitch_link.STL; visual mesh filename=package://pai_cl_12_240823/meshes/r_hip_pitch_link.STL
- link base_link: mass 1.28649761 -> 1.82
- link l_ankle_roll_link: mass 0.58347191 -> 0.58347
- link l_calf_link: mass 0.7182 -> 0.7601909
- link l_hip_roll_link: mass 0.3854 -> 0.41506
- link l_thigh_link: mass 0.074503 -> 0.12098061
- link r_ankle_pitch_link: mass 0.13223 -> 0.1322312
- link r_ankle_roll_link: mass 0.58347191 -> 0.58347
- link r_calf_link: mass 0.7282 -> 0.7601909
- link r_hip_roll_link: mass 0.3854 -> 0.41506
- link r_thigh_link: mass 0.07450262 -> 0.12098061
Joints:
- removed joint l_hip_yaw_joint
- removed joint r_hip_yaw_joint
- added joint l_hip_pitch_joint: type revolute, parent base_link, child l_hip_pitch_link, origin xyz=-0.0028186 0.0482 -0.031 rpy=0 0 0, axis 0 1 0, limit lower=-3.14 upper=3.14 effort=21 velocity=21
- added joint r_hip_pitch_joint: type revolute, parent base_link, child r_hip_pitch_link, origin xyz=-0.0028186 -0.0482 -0.031 rpy=0 0 0, axis 0 1 0, limit lower=-3.14 upper=3.14 effort=21 velocity=21
- joint l_hip_roll_joint: parent l_hip_yaw_link -> l_hip_pitch_link
- joint r_hip_roll_joint: parent r_hip_yaw_link -> r_hip_pitch_link

Commit message: 0910

File: urdf/pai_cl_12_240823.urdf (robot description, URDF)
Before this commit: robot pai_cl_12_240823, 13 links, 12 joints
Links:
- added link base_trunk, mass 1.82; collision box size=0.1 0.1 0.1; visual mesh filename=package://pai_cl_12_240823/meshes/base_link.STL
- link base_link: mass 1.82 -> None; geometry 
- link l_ankle_pitch_link: geometry collision box size=0.001 0.001 0.001; visual mesh filename=package://pai_cl_12_240823/meshes/l_ankle_pitch_link.STL
- link l_calf_link: geometry collision box size=0.001 0.001 0.001; visual mesh filename=package://pai_cl_12_240823/meshes/l_calf_link.STL
- link l_hip_pitch_link: geometry collision box size=0.001 0.001 0.001; visual mesh filename=package://pai_cl_12_240823/meshes/l_hip_pitch_link.STL
- link l_hip_roll_link: geometry collision box size=0.001 0.001 0.001; visual mesh filename=package://pai_cl_12_240823/meshes/l_hip_roll_link.STL
- link l_thigh_link: geometry collision box size=0.001 0.001 0.001; visual mesh filename=package://pai_cl_12_240823/meshes/l_thigh_link.STL
- link r_ankle_pitch_link: geometry collision box size=0.001 0.001 0.001; visual mesh filename=package://pai_cl_12_240823/meshes/r_ankle_pitch_link.STL
- link r_calf_link: geometry collision box size=0.001 0.001 0.001; visual mesh filename=package://pai_cl_12_240823/meshes/r_calf_link.STL
- link r_hip_pitch_link: geometry collision box size=0.001 0.001 0.001; visual mesh filename=package://pai_cl_12_240823/meshes/r_hip_pitch_link.STL
- link r_hip_roll_link: geometry collision box size=0.001 0.001 0.001; visual mesh filename=package://pai_cl_12_240823/meshes/r_hip_roll_link.STL
- link r_thigh_link: geometry collision box size=0.001 0.001 0.001; visual mesh filename=package://pai_cl_12_240823/meshes/r_thigh_link.STL
Joints:
- added joint base_joint: type fixed, parent base_link, child base_trunk, origin xyz=0.0 0.0 0.0 rpy=0.0 0.55 0.0, axis 0.0 0.0 0.0, limit lower=0.0 upper=0.0 effort=0.0 velocity=0.0
- joint l_ankle_pitch_joint: limit lower=-3.14 upper=3.14 effort=21 velocity=21 -> lower=-0.5 upper=0.7 effort=21 velocity=21
- joint l_ankle_roll_joint: limit lower=-3.14 upper=3.14 effort=21 velocity=21 -> lower=-0.8 upper=0.3 effort=21 velocity=21
- joint l_calf_joint: limit lower=-3.14 upper=3.14 effort=21 velocity=21 -> lower=0.0 upper=2.0 effort=21 velocity=21
- joint l_hip_pitch_joint: limit lower=-3.14 upper=3.14 effort=21 velocity=21 -> lower=-1.5 upper=1.5 effort=21 velocity=21; parent base_link -> base_trunk
- joint l_hip_roll_joint: limit lower=-3.14 upper=3.14 effort=21 velocity=21 -> lower=-0.12 upper=0.5 effort=21 velocity=21
- joint l_thigh_joint: limit lower=-3.14 upper=3.14 effort=21 velocity=21 -> lower=-0.3 upper=0.6 effort=21 velocity=21
- joint r_ankle_pitch_joint: limit lower=-3.14 upper=3.14 effort=21 velocity=21 -> lower=-0.5 upper=0.7 effort=21 velocity=21
- joint r_ankle_roll_joint: limit lower=-3.14 upper=3.14 effort=21 velocity=21 -> lower=-0.3 upper=0.8 effort=21 velocity=21
- joint r_calf_joint: limit lower=-3.14 upper=3.14 effort=21 velocity=21 -> lower=0.0 upper=2.0 effort=21 velocity=21
- joint r_hip_pitch_joint: limit lower=-3.14 upper=3.14 effort=21 velocity=21 -> lower=-1.5 upper=1.5 effort=21 velocity=21; parent base_link -> base_trunk
- joint r_hip_roll_joint: limit lower=-3.14 upper=3.14 effort=21 velocity=21 -> lower=-0.5 upper=0.12 effort=21 velocity=21
- joint r_thigh_joint: limit lower=-3.14 upper=3.14 effort=21 velocity=21 -> lower=-0.6 upper=0.3 effort=21 velocity=21
