Commit message: release 20241008

File: urdf/pi_12dof_release_v1.urdf (robot description, URDF)
Before this commit: robot clpai_12dof_0905, 13 links, 12 joints
Links:
- link base_link: geometry collision box size=0.1 0.1 0.1; visual mesh filename=package://pi_12dof_release_v1/meshes/baselink_1.STL
- link l_ankle_pitch_link: geometry collision box size=0.001 0.001 0.001; visual mesh filename=package://pi_12dof_release_v1/meshes/l_ankle_pitch_link.STL
- link l_ankle_roll_link: geometry collision mesh filename=package://pi_12dof_release_v1/meshes/l_ankle_roll_link.STL; visual mesh filename=package://pi_12dof_release_v1/meshes/l_ankle_roll_link.STL
- link l_calf_link: geometry collision box size=0.001 0.001 0.001; visual mesh filename=package://pi_12dof_release_v1/meshes/l_calf_link.STL
- link l_hip_pitch_link: geometry collision box size=0.001 0.001 0.001; visual mesh filename=package://pi_12dof_release_v1/meshes/l_hip_pitch_link.STL
- link l_hip_roll_link: geometry collision box size=0.001 0.001 0.001; visual mesh filename=package://pi_12dof_release_v1/meshes/l_hip_roll_link.STL
- link l_thigh_link: geometry collision box size=0.001 0.001 0.001; visual mesh filename=package://pi_12dof_release_v1/meshes/l_thigh_link.STL
- link r_ankle_pitch_link: geometry collision box size=0.001 0.001 0.001; visual mesh filename=package://pi_12dof_release_v1/meshes/r_ankle_pitch_link.STL
- link r_ankle_roll_link: geometry collision mesh filename=package://pi_12dof_release_v1/meshes/r_ankle_roll_link.STL; visual mesh filename=package://pi_12dof_release_v1/meshes/r_ankle_roll_link.STL
- link r_calf_link: geometry collision box size=0.001 0.001 0.001; visual mesh filename=package://pi_12dof_release_v1/meshes/r_calf_link.STL
- link r_hip_pitch_link: geometry collision box size=0.001 0.001 0.001; visual mesh filename=package://pi_12dof_release_v1/meshes/r_hip_pitch_link.STL
- link r_hip_roll_link: geometry collision box size=0.001 0.001 0.001; visual mesh filename=package://pi_12dof_release_v1/meshes/r_hip_roll_link.STL
- link r_thigh_link: geometry collision box size=0.001 0.001 0.001; visual mesh filename=package://pi_12dof_release_v1/meshes/r_thigh_link.STL
