Commit message: 241008

File: urdf/pi_parallel_12dof_release_v1.urdf (robot description, URDF)
Before this commit: robot pai_12dof_0911, 13 links, 12 joints
Links:
- link base_link: geometry collision box size=0.1 0.1 0.1; visual mesh filename=package://pi_parallel_12dof_release_v1/meshes/base_link.STL
- link l_ankle_pitch_link: geometry collision mesh filename=package://pi_parallel_12dof_release_v1/meshes/l_ankle_pitch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; visual mesh filename=package://pi_parallel_12dof_release_v1/meshes/l_ankle_pitch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
- link l_ankle_roll_link: geometry collision mesh filename=package://pi_parallel_12dof_release_v1/meshes/l_ankle_roll_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; visual mesh filename=package://pi_parallel_12dof_release_v1/meshes/l_ankle_roll_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
- link l_calf_link: geometry collision box size=0.04 0.04 0.10; visual mesh filename=package://pi_parallel_12dof_release_v1/meshes/l_calf_link.S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
- link l_hip_roll_link: geometry collision box size=0.03 0.03 0.03; visual mesh filename=package://pi_parallel_12dof_release_v1/meshes/l_hip_roll_li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
- link l_hip_yaw_link: geometry collision box size=0.03 0.03 0.03; visual mesh filename=package://pi_parallel_12dof_release_v1/meshes/l_hip_yaw_lin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
- link l_thigh_link: geometry collision box size=0.03 0.03 0.10; visual mesh filename=package://pi_parallel_12dof_release_v1/meshes/l_thigh_link.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
- link r_ankle_pitch_link: geometry collision mesh filename=package://pi_parallel_12dof_release_v1/meshes/r_ankle_pitch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; visual mesh filename=package://pi_parallel_12dof_release_v1/meshes/r_ankle_pitch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
- link r_ankle_roll_link: geometry collision mesh filename=package://pi_parallel_12dof_release_v1/meshes/r_ankle_roll_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; visual mesh filename=package://pi_parallel_12dof_release_v1/meshes/r_ankle_roll_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
- link r_calf_link: geometry collision box size=0.04 0.04 0.10; visual mesh filename=package://pi_parallel_12dof_release_v1/meshes/r_calf_link.S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
- link r_hip_roll_link: geometry collision box size=0.03 0.03 0.03; visual mesh filename=package://pi_parallel_12dof_release_v1/meshes/r_hip_roll_li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
- link r_hip_yaw_link: geometry collision box size=0.03 0.03 0.03; visual mesh filename=package://pi_parallel_12dof_release_v1/meshes/r_hip_yaw_lin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
- link r_thigh_link: geometry collision box size=0.03 0.03 0.10; visual mesh filename=package://pi_parallel_12dof_release_v1/meshes/r_thigh_link.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
