Commit message: modify the zero point

File: pi_12dof/urdf/pi_12dof.urdf (robot description, URDF)
Before this commit: robot pi_description, 13 links, 12 joints
Links:
- link base_link: geometry collision box size=0.17 0.15 0.15; visual mesh filename=package://pi_12dof/meshes/baselink_1.STL
- link l_ankle_pitch_link: geometry collision box size=0.07 0.065 0.045; visual mesh filename=package://pi_12dof/meshes/l_ankle_pitch_link.STL
- link l_ankle_roll_link: geometry collision mesh filename=package://pi_12dof/meshes/foot.STL scale=0.001 0.001 0.001; visual mesh filename=package://pi_12dof/meshes/l_ankle_roll_link.STL
- link l_calf_link: geometry collision box size=0.001 0.001 0.001; visual mesh filename=package://pi_12dof/meshes/l_calf_link.STL
- link l_hip_pitch_link: geometry collision box size=0.001 0.001 0.001; visual mesh filename=package://pi_12dof/meshes/l_hip_pitch_link.STL
- link l_hip_roll_link: geometry collision box size=0.001 0.001 0.001; visual mesh filename=package://pi_12dof/meshes/l_hip_roll_link.STL
- link l_thigh_link: geometry collision box size=0.001 0.001 0.001; visual mesh filename=package://pi_12dof/meshes/l_thigh_link.STL
- link r_ankle_pitch_link: geometry collision box size=0.07 0.065 0.045; visual mesh filename=package://pi_12dof/meshes/r_ankle_pitch_link.STL
- link r_ankle_roll_link: geometry collision mesh filename=package://pi_12dof/meshes/foot.STL scale=0.001 0.001 0.001; visual mesh filename=package://pi_12dof/meshes/r_ankle_roll_link.STL
- link r_calf_link: geometry collision box size=0.001 0.001 0.001; visual mesh filename=package://pi_12dof/meshes/r_calf_link.STL
- link r_hip_pitch_link: geometry collision box size=0.001 0.001 0.001; visual mesh filename=package://pi_12dof/meshes/r_hip_pitch_link.STL
- link r_hip_roll_link: geometry collision box size=0.001 0.001 0.001; visual mesh filename=package://pi_12dof/meshes/r_hip_roll_link.STL
- link r_thigh_link: geometry collision box size=0.001 0.001 0.001; visual mesh filename=package://pi_12dof/meshes/r_thigh_link.STL
Joints:
- joint l_ankle_pitch_joint: origin xyz=0 0 -0.14 rpy=0 -0.4 0 -> xyz=0 0 -0.14 rpy=0 0 0
- joint l_calf_joint: origin xyz=0 0 -0.07025 rpy=0 0.65 0 -> xyz=0 0 -0.07025 rpy=0 0 0
- joint l_hip_pitch_joint: origin xyz=-5.1979E-05 0.0233 -0.033 rpy=0 -0.25 0 -> xyz=-5.1979E-05 0.0233 -0.033 rpy=0 0 0
- joint r_ankle_pitch_joint: origin xyz=0 0 -0.14 rpy=0 -0.4 0 -> xyz=0 0 -0.14 rpy=0 0 0
- joint r_calf_joint: origin xyz=0 -0.0027 -0.07025 rpy=0 0.65 0 -> xyz=0 -0.0027 -0.07025 rpy=0 0 0
- joint r_hip_pitch_joint: origin xyz=-5.1979E-05 -0.0233 -0.033 rpy=0 -0.25 0 -> xyz=-5.1979E-05 -0.0233 -0.033 rpy=0 0 0
