Commit message: fix name of link and meshs

File: hi_23dof/urdf/hi_23dof.urdf (robot description, URDF)
Before this commit: robot hi_25dof, 26 links, 25 joints
Links:
- link base_link: geometry collision mesh filename=package://hi_23dof/meshes/base_link.STL; visual mesh filename=package://hi_23dof/meshes/base_link.STL
- link head_pitch_link: geometry collision mesh filename=package://hi_23dof/meshes/head_pitch_link.STL; visual mesh filename=package://hi_23dof/meshes/head_pitch_link.STL
- link head_yaw_link: geometry collision mesh filename=package://hi_23dof/meshes/head_yaw_link.STL; visual mesh filename=package://hi_23dof/meshes/head_yaw_link.STL
- link l_ankle_pitch_Link: geometry collision mesh filename=package://hi_23dof/meshes/l_ankle_pitch_Link.STL; visual mesh filename=package://hi_23dof/meshes/l_ankle_pitch_Link.STL
- link l_ankle_roll_Link: geometry collision mesh filename=package://hi_23dof/meshes/l_ankle_roll_Link.STL; visual mesh filename=package://hi_23dof/meshes/l_ankle_roll_Link.STL
- link l_elbow_link: geometry collision mesh filename=package://hi_23dof/meshes/l_elbow_link.STL; visual mesh filename=package://hi_23dof/meshes/l_elbow_link.STL
- link l_hip_calf_Link: geometry collision mesh filename=package://hi_23dof/meshes/l_hip_calf_Link.STL; visual mesh filename=package://hi_23dof/meshes/l_hip_calf_Link.STL
- link l_hip_pitch_link: geometry collision mesh filename=package://hi_23dof/meshes/l_hip_pitch_link.STL; visual mesh filename=package://hi_23dof/meshes/l_hip_pitch_link.STL
- link l_hip_roll_Link: geometry collision mesh filename=package://hi_23dof/meshes/l_hip_roll_Link.STL; visual mesh filename=package://hi_23dof/meshes/l_hip_roll_Link.STL
- link l_hip_thigh_Link: geometry collision mesh filename=package://hi_23dof/meshes/l_hip_thigh_Link.STL; visual mesh filename=package://hi_23dof/meshes/l_hip_thigh_Link.STL
- link l_shoulder_pitch_link: geometry collision mesh filename=package://hi_23dof/meshes/l_shoulder_pitch_link.STL; visual mesh filename=package://hi_23dof/meshes/l_shoulder_pitch_link.STL
- link l_shoulder_roll_link: geometry collision mesh filename=package://hi_23dof/meshes/l_shoulder_roll_link.STL; visual mesh filename=package://hi_23dof/meshes/l_shoulder_roll_link.STL
- link l_upper_arm_link: geometry collision mesh filename=package://hi_23dof/meshes/l_upper_arm_link.STL; visual mesh filename=package://hi_23dof/meshes/l_upper_arm_link.STL
- link l_wrist_link: geometry collision mesh filename=package://hi_23dof/meshes/l_wrist_link.STL; visual mesh filename=package://hi_23dof/meshes/l_wrist_link.STL
- link r_ankle_pitch_link: geometry collision mesh filename=package://hi_23dof/meshes/r_ankle_pitch_link.STL; visual mesh filename=package://hi_23dof/meshes/r_ankle_pitch_link.STL
- link r_ankle_roll_link: geometry collision mesh filename=package://hi_23dof/meshes/r_ankle_roll_link.STL; visual mesh filename=package://hi_23dof/meshes/r_ankle_roll_link.STL
- link r_elbow_link: geometry collision mesh filename=package://hi_23dof/meshes/r_elbow_link.STL; visual mesh filename=package://hi_23dof/meshes/r_elbow_link.STL
- link r_hip_calf_link: geometry collision mesh filename=package://hi_23dof/meshes/r_hip_calf_link.STL; visual mesh filename=package://hi_23dof/meshes/r_hip_calf_link.STL
- link r_hip_pitch_Link: geometry collision mesh filename=package://hi_23dof/meshes/r_hip_pitch_Link.STL; visual mesh filename=package://hi_23dof/meshes/r_hip_pitch_Link.STL
- link r_hip_roll_Link: geometry collision mesh filename=package://hi_23dof/meshes/r_hip_roll_Link.STL; visual mesh filename=package://hi_23dof/meshes/r_hip_roll_Link.STL
- link r_hip_thigh_link: geometry collision mesh filename=package://hi_23dof/meshes/r_hip_thigh_link.STL; visual mesh filename=package://hi_23dof/meshes/r_hip_thigh_link.STL
- link r_shoulder_pitch_link: geometry collision mesh filename=package://hi_23dof/meshes/r_shoulder_pitch_link.STL; visual mesh filename=package://hi_23dof/meshes/r_shoulder_pitch_link.STL
- link r_shoulder_roll_link: geometry collision mesh filename=package://hi_23dof/meshes/r_shoulder_roll_link.STL; visual mesh filename=package://hi_23dof/meshes/r_shoulder_roll_link.STL
- link r_upper_arm_link: geometry collision mesh filename=package://hi_23dof/meshes/r_upper_arm_link.STL; visual mesh filename=package://hi_23dof/meshes/r_upper_arm_link.STL
- link r_wrist_link: geometry collision mesh filename=package://hi_23dof/meshes/r_wrist_link.STL; visual mesh filename=package://hi_23dof/meshes/r_wrist_link.STL
- link waist_yaw_link: geometry collision mesh filename=package://hi_23dof/meshes/waist_yaw_link.STL; visual mesh filename=package://hi_23dof/meshes/waist_yaw_link.STL
Joints:
- removed joint head_pitch_joint
- removed joint head_yaw_joint
