Commit message: add hi_25dof.xml

File: hi_25dof/urdf/hi_25dof.urdf (robot description, URDF)
Before this commit: robot hi_25dof, 26 links, 25 joints
Links:
- removed link l_hip_caif_Link
- removed link r_hip_caif_Link
- added link l_hip_calf_Link, mass 1.6427; collision mesh filename=package://hi_25dof/meshes/l_hip_calf_Link.STL; visual mesh filename=package://hi_25dof/meshes/l_hip_calf_Link.STL
- added link r_hip_calf_Link, mass 1.6427; collision mesh filename=package://hi_25dof/meshes/r_hip_calf_Link.STL; visual mesh filename=package://hi_25dof/meshes/r_hip_calf_Link.STL
- added link world
Joints:
- removed joint l_hip_caif_joint
- removed joint r_hip_caif_joint
- added joint floating_base_joint: type floating, parent world, child base_link
- added joint l_hip_calf_joint: type revolute, parent l_hip_thigh_Link, child l_hip_calf_Link, origin xyz=0 0.00375 -0.097 rpy=0 0 0, axis 0 1 0, limit lower=-1.5708 upper=2.0944 effort=32.4 velocity=5.55
- added joint r_hip_calf_joint: type revolute, parent r_hip_thigh_Link, child r_hip_calf_Link, origin xyz=0 -0.00375 -0.097 rpy=0 0 0, axis 0 1 0, limit lower=-1.5708 upper=2.0944 effort=32.4 velocity=5.55
- joint l_ankle_pitch_joint: parent l_hip_caif_Link -> l_hip_calf_Link
- joint r_ankle_pitch_joint: parent r_hip_caif_Link -> r_hip_calf_Link

Commit message: fixed pi mass

File: hi_25dof/urdf/hi_25dof.urdf (robot description, URDF)
Before this commit: robot hi_25dof, 27 links, 26 joints
Links:
- removed link world
Joints:
- removed joint floating_base_joint

File: pi_12dof/urdf/pi_12dof.urdf (robot description, URDF)
Before this commit: robot pi_description, 13 links, 12 joints
Links:
- link base_link: mass 2.1609 -> 1.94350955
- link l_ankle_pitch_link: mass 0.1759244 ->  0.16558271
- link l_ankle_roll_link: mass 0.51868476 -> 0.62234851
- link l_calf_link: mass 0.81374212 -> 0.80286993
- link l_hip_pitch_link: mass 0.38968624 -> 0.39857633; geometry collision box size=0.05 0.05 0.05; visual mesh filename=package://pi_12dof/meshes/l_hip_pitch_link.STL
- link l_hip_roll_link: mass 0.38851552 -> 0.48571832
- link l_thigh_link: mass 0.11270879 ->  0.10937966
- link r_ankle_pitch_link: mass 0.1759244 -> 0.16558271
- link r_ankle_roll_link: mass 0.51868476 -> 0.62234851
- link r_calf_link: mass 0.81374212 -> 0.80286993
- link r_hip_pitch_link: mass 0.36999771 ->  0.39857633; geometry collision box size=0.05 0.05 0.05; visual mesh filename=package://pi_12dof/meshes/r_hip_pitch_link.STL
- link r_hip_roll_link: mass 0.38851552 -> 0.48571832
- link r_thigh_link: mass 0.11270879 -> 0.10937966
Joints:
- removed joint l_ankle_pitch_joint
- removed joint l_ankle_roll_joint
- removed joint l_calf_joint
- removed joint l_hip_pitch_joint
- removed joint l_hip_roll_joint
- removed joint l_thigh_joint
- removed joint r_ankle_pitch_joint
- removed joint r_ankle_roll_joint
- removed joint r_calf_joint
- removed joint r_hip_pitch_joint
- removed joint r_hip_roll_joint
- removed joint r_thigh_joint
- added joint 01_r_hip_pitch_joint: type revolute, parent base_link, child r_hip_pitch_link, origin xyz=-5.1979E-05 -0.0233 -0.033 rpy=0 0 0, axis 0 1 0, limit lower=-1.5 upper=1.5 effort=20 velocity=5.45
- added joint 02_r_hip_roll_joint: type revolute, parent r_hip_pitch_link, child r_hip_roll_link, origin xyz=0.00025 -0.0568 0 rpy=0 0 0, axis 1 0 0, limit lower=-0.38 upper=1.2 effort=20 velocity=5.45
- added joint 03_r_thigh_joint: type revolute, parent r_hip_roll_link, child r_thigh_link, origin xyz=-0.00025 0 -0.06925 rpy=0 0 0, axis 0 0 1, limit lower=-1 upper=1 effort=20 velocity=5.45
- added joint 04_r_calf_joint: type revolute, parent r_thigh_link, child r_calf_link, origin xyz=0 -0.0027 -0.07025 rpy=0 0 0, axis 0 1 0, limit lower=0 upper=2.2 effort=20 velocity=5.45
- added joint 05_r_ankle_pitch_joint: type revolute, parent r_calf_link, child r_ankle_pitch_link, origin xyz=0 0 -0.14 rpy=0 0 0, axis 0 1 0, limit lower=-0.8 upper=0.8 effort=20 velocity=5.45
- added joint 06_r_ankle_roll_joint: type revolute, parent r_ankle_pitch_link, child r_ankle_roll_link, origin xyz=0.07525 0.0027 0 rpy=0 0 0, axis 1 0 0, limit lower=-0.6 upper=0.6 effort=20 velocity=5.45
- added joint 07_l_hip_pitch_joint: type revolute, parent base_link, child l_hip_pitch_link, origin xyz=-5.1979E-05 0.0233 -0.033 rpy=0 0 0, axis 0 1 0, limit lower=-1.5 upper=1.5 effort=20 velocity=5.45
- added joint 08_l_hip_roll_joint: type revolute, parent l_hip_pitch_link, child l_hip_roll_link, origin xyz=0 0.0568 0 rpy=0 0 0, axis 1 0 0, limit lower=-0.38 upper=1.2 effort=20 velocity=5.45
- added joint 09_l_thigh_joint: type revolute, parent l_hip_roll_link, child l_thigh_link, origin xyz=0 0 -0.06925 rpy=0 0 0, axis 0 0 1, limit lower=-1 upper=1 effort=20 velocity=5.45
- added joint 10_l_calf_joint: type revolute, parent l_thigh_link, child l_calf_link, origin xyz=0 0 -0.07025 rpy=0 0 0, axis 0 1 0, limit lower=0 upper=2.2 effort=20 velocity=5.45
- added joint 11_l_ankle_pitch_joint: type revolute, parent l_calf_link, child l_ankle_pitch_link, origin xyz=0 0 -0.14 rpy=0 0 0, axis 0 1 0, limit lower=-0.8 upper=0.8 effort=20 velocity=5.45
- added joint 12_l_ankle_roll_joint: type revolute, parent l_ankle_pitch_link, child l_ankle_roll_link, origin xyz=0.07525 0 0 rpy=0 0 0, axis 1 0 0, limit lower=-0.6 upper=0.6 effort=20 velocity=5.45

Commit message: fix hi urdf

File: hi_25dof/urdf/hi_25dof.urdf (robot description, URDF)
Before this commit: robot hi_25dof, 26 links, 25 joints
Links:
- removed link l_ankle_pitch_Link
- removed link l_ankle_roll_Link
- removed link l_hip_calf_Link
- removed link l_hip_thigh_Link
- removed link r_hip_pitch_Link
- removed link r_hip_roll_Link
- added link l_ankle_pitch_link, mass 0.056538; collision box size=0.01 0.01 0.01; visual mesh filename=package://hi_25dof/meshes/l_ankle_pitch_link.STL
- added link l_ankle_roll_link, mass 0.59911; collision mesh filename=package://hi_25dof/meshes/l_ankle_roll_link.STL; visual mesh filename=package://hi_25dof/meshes/l_ankle_roll_link.STL
- added link l_hip_calf_link, mass 1.6427; collision box size=0.06 0.06 0.21; visual mesh filename=package://hi_25dof/meshes/l_hip_calf_link.STL
- added link l_hip_thigh_link, mass 0.24756; collision box size=0.01 0.01 0.01; visual mesh filename=package://hi_25dof/meshes/l_hip_thigh_link.STL
- added link r_hip_pitch_link, mass 0.66505; collision box size=0.06 0.07 0.06; visual mesh filename=package://hi_25dof/meshes/r_hip_pitch_link.STL
- added link r_hip_roll_link, mass 0.78331; collision box size=0.06 0.07 0.06; visual mesh filename=package://hi_25dof/meshes/r_hip_roll_link.STL
- link base_link: geometry collision box size=0.12 0.2 0.22; visual mesh filename=package://hi_25dof/meshes/base_link.STL
- link head_pitch_link: geometry collision box size=0.1 0.15 0.03; visual mesh filename=package://hi_25dof/meshes/head_pitch_link.STL
- link head_yaw_link: geometry collision box size=0.03 0.03 0.03; visual mesh filename=package://hi_25dof/meshes/head_yaw_link.STL
- link l_elbow_link: geometry collision box size=0.05 0.05 0.05; visual mesh filename=package://hi_25dof/meshes/l_elbow_link.STL
- link l_hip_pitch_link: geometry collision box size=0.06 0.07 0.06; visual mesh filename=package://hi_25dof/meshes/l_hip_pitch_link.STL
- link l_hip_roll_Link: geometry collision box size=0.06 0.07 0.06; visual mesh filename=package://hi_25dof/meshes/l_hip_roll_Link.STL
- link l_shoulder_pitch_link: geometry collision box size=0.05 0.05 0.05; visual mesh filename=package://hi_25dof/meshes/l_shoulder_pitch_link.STL
- link l_shoulder_roll_link: geometry collision box size=0.05 0.05 0.05; visual mesh filename=package://hi_25dof/meshes/l_shoulder_roll_link.STL
- link l_upper_arm_link: geometry collision box size=0.05 0.05 0.05; visual mesh filename=package://hi_25dof/meshes/l_upper_arm_link.STL
- link l_wrist_link: geometry collision box size=0.02 0.02 0.05; visual mesh filename=package://hi_25dof/meshes/l_wrist_link.STL
- link r_ankle_pitch_link: geometry collision box size=0.01 0.01 0.01; visual mesh filename=package://hi_25dof/meshes/r_ankle_pitch_link.STL
- link r_elbow_link: geometry collision box size=0.05 0.05 0.05; visual mesh filename=package://hi_25dof/meshes/r_elbow_link.STL
- link r_hip_calf_link: geometry collision box size=0.06 0.06 0.21; visual mesh filename=package://hi_25dof/meshes/r_hip_calf_link.STL
- link r_hip_thigh_link: geometry collision box size=0.01 0.01 0.01; visual mesh filename=package://hi_25dof/meshes/r_hip_thigh_link.STL
- link r_shoulder_pitch_link: geometry collision box size=0.05 0.05 0.05; visual mesh filename=package://hi_25dof/meshes/r_shoulder_pitch_link.STL
- link r_shoulder_roll_link: geometry collision box size=0.05 0.05 0.05; visual mesh filename=package://hi_25dof/meshes/r_shoulder_roll_link.STL
- link r_upper_arm_link: geometry collision box size=0.05 0.05 0.05; visual mesh filename=package://hi_25dof/meshes/r_upper_arm_link.STL
- link r_wrist_link: geometry collision box size=0.02 0.02 0.05; visual mesh filename=package://hi_25dof/meshes/r_wrist_link.STL
- link waist_yaw_link: geometry collision box size=0.09 0.07 0.09; visual mesh filename=package://hi_25dof/meshes/waist_yaw_link.STL
Joints:
- joint l_ankle_pitch_joint: child l_ankle_pitch_Link -> l_ankle_pitch_link; parent l_hip_calf_Link -> l_hip_calf_link
- joint l_ankle_roll_joint: child l_ankle_roll_Link -> l_ankle_roll_link; parent l_ankle_pitch_Link -> l_ankle_pitch_link
- joint l_hip_calf_joint: child l_hip_calf_Link -> l_hip_calf_link; parent l_hip_thigh_Link -> l_hip_thigh_link
- joint l_hip_thigh_joint: child l_hip_thigh_Link -> l_hip_thigh_link
- joint r_hip_pitch_joint: child r_hip_pitch_Link -> r_hip_pitch_link
- joint r_hip_roll_joint: child r_hip_roll_Link -> r_hip_roll_link; parent r_hip_pitch_Link -> r_hip_pitch_link
- joint r_hip_thigh_joint: parent r_hip_roll_Link -> r_hip_roll_link

Commit message: add collision

File: hi_25dof/urdf/hi_25dof.urdf (robot description, URDF)
Before this commit: robot hi_25dof, 26 links, 25 joints
Links:
- removed link l_hip_roll_Link
- added link l_hip_roll_link, mass 0.78331; collision box size=0.06 0.07 0.06; visual mesh filename=package://hi_25dof/meshes/l_hip_roll_link.STL
- link l_ankle_roll_link: geometry collision mesh filename=package://hi_25dof/meshes/ankle_roll_simplify.STL scale=0.001 0.001 0.001; visual mesh filename=package://hi_25dof/meshes/l_ankle_roll_link.STL
- link l_elbow_link: geometry collision box size=0.04 0.04 0.04; visual mesh filename=package://hi_25dof/meshes/l_elbow_link.STL
- link l_wrist_link: geometry collision box size=0.02 0.02 0.025; collision sphere radius=0.0175
- link r_ankle_roll_link: geometry collision mesh filename=package://hi_25dof/meshes/ankle_roll_simplify.STL scale=0.001 0.001 0.001; visual mesh filename=package://hi_25dof/meshes/r_ankle_roll_link.STL
- link r_elbow_link: geometry collision box size=0.04 0.04 0.04; visual mesh filename=package://hi_25dof/meshes/r_elbow_link.STL
- link r_wrist_link: geometry collision box size=0.02 0.02 0.025; collision sphere radius=0.0175
- link waist_yaw_link: geometry collision box size=0.09 0.07 0.05; visual mesh filename=package://hi_25dof/meshes/waist_yaw_link.STL
Joints:
- joint l_hip_roll_joint: child l_hip_roll_Link -> l_hip_roll_link
- joint l_hip_thigh_joint: parent l_hip_roll_Link -> l_hip_roll_link

Commit message: fix collision

File: hi_25dof/urdf/hi_25dof.urdf (robot description, URDF)
Before this commit: robot hi_25dof, 26 links, 25 joints
Links:
- link base_link: geometry collision box size=0.05 0.1 0.065; visual mesh filename=package://hi_25dof/meshes/base_link.STL
- link waist_yaw_link: geometry collision box size=0.09 0.07 0.05; collision box size=0.12 0.2 0.21

Commit message: fix collision

File: hi_25dof/urdf/hi_25dof.urdf (robot description, URDF)
Before this commit: robot hi_25dof, 26 links, 25 joints
Links:
- link l_shoulder_pitch_link: geometry collision box size=0.05 0.06 0.05; visual mesh filename=package://hi_25dof/meshes/l_shoulder_pitch_link.STL
- link r_shoulder_pitch_link: geometry collision box size=0.05 0.06 0.05; visual mesh filename=package://hi_25dof/meshes/r_shoulder_pitch_link.STL
